File: PCBs/GPS Board/GPS Board Rev C.brd (EAGLE design)
At the start: 95.9 x 90.2 mm, 11 parts

Commit message: Improve decoupling, ground impedance, silkscreens
Parts:
- moved C2 0.13 mm to (66.7, 83.8)
Routing:
- net GND: track 5.72 -> 8.77 mm, vias 3 -> 6
- net SW9: track 131.9 -> 133.0 mm
Changed lines of the file:
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@@
 <setting verticaltext="up"/>
 </settings>
-<grid distance="25" unitdist="mil" unit="mil" style="lines" multiple="1" display="yes" altdistance="5" altunitdist="mil" altunit="mil"/>
+<grid distance="25" unitdist="mil" unit="mil" style="lines" multiple="1" display="yes" altdistance="2.5" altunitdist="mil" altunit="mil"/>
 <layers>
 <layer number="1" name="Top" color="4" fill="1" visible="yes" active="yes"/>
@@
 </autorouter>
 <elements>
-<element name="C2" library="resistor" library_urn="urn:adsk.eagle:library:348" package="C0805" package3d_urn="urn:adsk.eagle:package:26137/1" value="1uF" x="66.548" y="83.82" smashed="yes" rot="R270">
-<attribute name="NAME" x="65.5955" y="86.8045" size="1.016" layer="25"/>
-<attribute name="VALUE" x="65.786" y="85.979" size="0.635" layer="27"/>
+<element name="C2" library="resistor" library_urn="urn:adsk.eagle:library:348" package="C0805" package3d_urn="urn:adsk.eagle:package:26137/1" value="1uF" x="66.675" y="83.82" smashed="yes" rot="R270">
+<attribute name="NAME" x="65.7225" y="86.8045" size="1.016" layer="25"/>
+<attribute name="VALUE" x="65.913" y="85.979" size="0.635" layer="27"/>
 </element>
 <element name="C1" library="resistor" library_urn="urn:adsk.eagle:library:348" package="C0805" package3d_urn="urn:adsk.eagle:package:26137/1" value="0.1uF" x="64.135" y="83.82" smashed="yes" rot="R270">
@@
 </element>
 <element name="U$2" library="Cubesat" package="PC104_NO_DIMENSION" value="PC104_NO_DIMENSION" x="0" y="0"/>
-<element name="GND" library="testpad" library_urn="urn:adsk.eagle:library:385" package="TP10SQ" package3d_urn="urn:adsk.eagle:package:27962/1" value="TPTP10SQ" x="16.51" y="43.18">
-<attribute name="TP_SIGNAL_NAME" value="" x="16.51" y="43.18" size="1.778" layer="27" display="off"/>
-</element>
-<element name="TX" library="testpad" library_urn="urn:adsk.eagle:library:385" package="TP10SQ" package3d_urn="urn:adsk.eagle:package:27962/1" value="TPTP10SQ" x="16.51" y="46.99">
-<attribute name="TP_SIGNAL_NAME" value="" x="16.51" y="46.99" size="1.778" layer="27" display="off"/>
-</element>
-<element name="RX" library="testpad" library_urn="urn:adsk.eagle:library:385" package="TP10SQ" package3d_urn="urn:adsk.eagle:package:27962/1" value="TPTP10SQ" x="16.51" y="50.8">
-<attribute name="TP_SIGNAL_NAME" value="" x="16.51" y="50.8" size="1.778" layer="27" display="off"/>
-</element>
-<element name="3V3" library="testpad" library_urn="urn:adsk.eagle:library:385" package="TP10SQ" package3d_urn="urn:adsk.eagle:package:27962/1" value="TPTP10SQ" x="16.51" y="62.23">
-<attribute name="TP_SIGNAL_NAME" value="" x="16.51" y="62.23" size="1.778" layer="27" display="off"/>
-</element>
-<element name="VPP" library="testpad" library_urn="urn:adsk.eagle:library:385" package="TP10SQ" package3d_urn="urn:adsk.eagle:package:27962/1" value="TPTP10SQ" x="16.51" y="54.61">
-<attribute name="TP_SIGNAL_NAME" value="" x="16.51" y="54.61" size="1.778" layer="27" display="off"/>
-</element>
-<element name="PF" library="testpad" library_urn="urn:adsk.eagle:library:385" package="TP10SQ" package3d_urn="urn:adsk.eagle:package:27962/1" value="TPTP10SQ" x="16.51" y="58.42">
-<attribute name="TP_SIGNAL_NAME" value="" x="16.51" y="58.42" size="1.778" layer="27" display="off"/>
+<element name="GND" library="testpad" library_urn="urn:adsk.eagle:library:385" package="TP10SQ" package3d_urn="urn:adsk.eagle:package:27962/1" value="TPTP10SQ" x="16.51" y="43.18" smashed="yes">
+<attribute name="NAME" x="16.0099" y="43.7299" size="1.27" layer="25"/>
+<attribute name="TP_SIGNAL_NAME" value="" x="16.51" y="41.275" size="1" layer="37"/>
+</element>
+<element name="TX" library="testpad" library_urn="urn:adsk.eagle:library:385" package="TP10SQ" package3d_urn="urn:adsk.eagle:package:27962/1" value="TPTP10SQ" x="16.51" y="46.99" smashed="yes">
+<attribute name="NAME" x="16.0099" y="47.5399" size="1.27" layer="25"/>
+<attribute name="TP_SIGNAL_NAME" value="" x="16.51" y="45.085" size="1" layer="37"/>
+</element>
+<element name="RX" library="testpad" library_urn="urn:adsk.eagle:library:385" package="TP10SQ" package3d_urn="urn:adsk.eagle:package:27962/1" value="TPTP10SQ" x="16.51" y="50.8" smashed="yes">
+<attribute name="NAME" x="16.0099" y="51.3499" size="1.27" layer="25"/>
+<attribute name="TP_SIGNAL_NAME" value="" x="16.51" y="48.895" size="1" layer="37"/>
+</element>
+<element name="3V3" library="testpad" library_urn="urn:adsk.eagle:library:385" package="TP10SQ" package3d_urn="urn:adsk.eagle:package:27962/1" value="TPTP10SQ" x="16.51" y="62.23" smashed="yes">
+<attribute name="NAME" x="16.0099" y="62.7799" size="1.27" layer="25"/>
+<attribute name="TP_SIGNAL_NAME" value="" x="16.51" y="60.325" size="1" layer="37"/>
+</element>
+<element name="VPP" library="testpad" library_urn="urn:adsk.eagle:library:385" package="TP10SQ" package3d_urn="urn:adsk.eagle:package:27962/1" value="TPTP10SQ" x="16.51" y="54.61" smashed="yes">
+<attribute name="NAME" x="16.0099" y="55.1599" size="1.27" layer="25"/>
+<attribute name="TP_SIGNAL_NAME" value="" x="16.51" y="52.705" size="1" layer="37"/>
+</element>
+<element name="PF" library="testpad" library_urn="urn:adsk.eagle:library:385" package="TP10SQ" package3d_urn="urn:adsk.eagle:package:27962/1" value="TPTP10SQ" x="16.51" y="58.42" smashed="yes">
+<attribute name="NAME" x="16.0099" y="58.9699" size="1.27" layer="25"/>
+<attribute name="TP_SIGNAL_NAME" value="" x="16.51" y="56.515" size="1" layer="37"/>
 </element>
 <element name="PINAV-CONNECTOR" library="HLE-110-02-X-DV" package="HLE-110-02-X-DV-PE-BE" value="HLE-110-02-X-DVHLE-110-X-DV-PE-BA" x="44.535" y="72.39" smashed="yes">
@@
 <signal name="SW9">
 <wire x1="81.28" y1="54.61" x2="69.85" y2="66.04" width="0.2032" layer="1"/>
-<wire x1="69.85" y1="66.04" x2="69.85" y2="82.55" width="0.2032" layer="1"/>
-<wire x1="69.85" y1="82.55" x2="67.63" y2="84.77" width="0.2032" layer="1"/>
+<wire x1="69.85" y1="82.55" x2="69.85" y2="66.04" width="0.2032" layer="1"/>
 <wire x1="86.995" y1="54.61" x2="81.28" y2="54.61" width="0.2032" layer="1"/>
 <contactref element="U$2" pad="71"/>
@@
 <contactref element="PINAV-CONNECTOR" pad="P$8"/>
 <contactref element="3V3" pad="TP"/>
-<wire x1="66.548" y1="84.77" x2="64.135" y2="84.77" width="0.508" layer="1"/>
+<wire x1="66.675" y1="84.77" x2="64.135" y2="84.77" width="0.508" layer="1"/>
 <wire x1="64.135" y1="84.77" x2="44.535" y2="84.77" width="0.508" layer="1"/>
 <wire x1="44.535" y1="84.77" x2="44.45" y2="84.77" width="0.2032" layer="1"/>
@@
 <wire x1="48.345" y1="76.2" x2="48.345" y2="80.875" width="0.508" layer="1"/>
 <wire x1="48.345" y1="80.875" x2="44.45" y2="84.77" width="0.508" layer="1"/>
-<wire x1="66.548" y1="84.77" x2="67.63" y2="84.77" width="0" layer="19" extent="1-1"/>
+<wire x1="66.675" y1="84.77" x2="67.63" y2="84.77" width="0.2032" layer="1"/>
+<wire x1="67.63" y1="84.77" x2="69.85" y2="82.55" width="0.2032" layer="1"/>
 </signal>
 <signal name="GND">
@@
 <contactref element="U$2" pad="99"/>
 <contactref element="GND" pad="TP"/>
-<wire x1="16.51" y1="43.18" x2="19.05" y2="43.18" width="0.2032" layer="1"/>
-<via x="19.05" y="43.18" extent="1-16" drill="0.254"/>
-<wire x1="64.135" y1="82.87" x2="64.135" y2="81.28" width="0.508" layer="1"/>
-<via x="64.135" y="81.28" extent="1-16" drill="0.254"/>
-<wire x1="66.548" y1="82.87" x2="66.548" y2="81.28" width="0.508" layer="1"/>
-<via x="66.548" y="81.28" extent="1-16" drill="0.254"/>
+<wire x1="16.51" y1="43.18" x2="17.526" y2="43.18" width="0.2032" layer="1"/>
+<via x="17.526" y="43.18" extent="1-16" drill="0.254"/>
+<wire x1="64.135" y1="82.87" x2="64.135" y2="81.534" width="0.508" layer="1"/>
+<via x="64.135" y="81.534" extent="1-16" drill="0.254"/>
+<wire x1="66.675" y1="82.87" x2="66.675" y2="81.534" width="0.508" layer="1"/>
+<via x="66.675" y="81.534" extent="1-16" drill="0.254"/>
+<via x="65.405" y="82.8675" extent="1-16" drill="0.254"/>
+<wire x1="65.405" y1="82.8675" x2="66.6725" y2="82.8675" width="0.508" layer="1"/>
+<wire x1="66.6725" y1="82.8675" x2="66.675" y2="82.87" width="0.508" layer="1"/>
+<wire x1="65.405" y1="82.8675" x2="64.1375" y2="82.8675" width="0.508" layer="1"/>
+<wire x1="64.1375" y1="82.8675" x2="64.135" y2="82.87" width="0.508" layer="1"/>
+<wire x1="66.675" y1="82.87" x2="67.9425" y2="82.87" width="0.508" layer="1"/>
+<wire x1="67.9425" y1="82.87" x2="67.945" y2="82.8675" width="0.508" layer="1"/>
+<via x="67.945" y="82.8675" extent="1-16" drill="0.254"/>
+<wire x1="64.135" y1="82.87" x2="62.8675" y2="82.87" width="0.508" layer="1"/>
+<wire x1="62.8675" y1="82.87" x2="62.865" y2="82.8675" width="0.508" layer="1"/>
+<via x="62.865" y="82.8675" extent="1-16" drill="0.254"/>
 </signal>
 <signal name="VPP">
