File: PCBs/Communication Board/Communication Board Rev A.brd (EAGLE design)
At the start: 95.9 x 90.2 mm, 22 parts

Commit message: Create comm parts list
Parts:
- removed THERM: TPSQTP20SQ, testpad:TP20SQ
- added R2: 0, resistor:R0805
- C2: value 47uF -> 10uF
Connections:
- net GND: now also R2.2
- net MNT1: now also R2.1; no longer THERM.TP
Routing:
- net GND: track 22.0 -> 23.7 mm, vias 8 -> 9
Other:
- board text added: "VT VCC Communication Board Rev A - 8/03/18"
- board text removed: "VT VCC Communication Board Rev A - 8/02/18"
Changed lines of the file:
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@@
 <?xml version="1.0" encoding="utf-8"?>
 <!DOCTYPE eagle SYSTEM "eagle.dtd">
-<eagle version="9.1.1">
+<eagle version="9.1.2">
 <drawing>
 <settings>
@@
 <wire x1="32.385" y1="90.17" x2="90.805" y2="90.17" width="0.2032" layer="20"/>
 <text x="79.375" y="89.535" size="1.778" layer="48" rot="R180">VT VCC Communication Board
-Rev A - 8/02/18</text>
+Rev A - 8/03/18</text>
 <rectangle x1="33.569275" y1="80.686275" x2="33.581975" y2="80.692625" layer="200"/>
 <rectangle x1="33.569275" y1="80.692625" x2="33.581975" y2="80.698975" layer="200"/>
@@
 <param name="rlMinPadBottom" value="7mil"/>
 <param name="rlMaxPadBottom" value="20mil"/>
-<param name="rlMinViaOuter" value="5mil"/>
+<param name="rlMinViaOuter" value="7mil"/>
 <param name="rlMaxViaOuter" value="20mil"/>
-<param name="rlMinViaInner" value="5mil"/>
+<param name="rlMinViaInner" value="7mil"/>
 <param name="rlMaxViaInner" value="20mil"/>
 <param name="rlMinMicroViaOuter" value="4mil"/>
@@
 <attribute name="VALUE" x="41.275" y="29.845" size="1.016" layer="27"/>
 </element>
-<element name="C2" library="resistor" library_urn="urn:adsk.eagle:library:348" package="C0805" package3d_urn="urn:adsk.eagle:package:23617/2" value="47uF" x="42.418" y="66.421" smashed="yes" rot="R90">
+<element name="C2" library="resistor" library_urn="urn:adsk.eagle:library:348" package="C0805" package3d_urn="urn:adsk.eagle:package:23617/2" value="10uF" x="42.418" y="66.421" smashed="yes" rot="R90">
 <attribute name="NAME" x="44.7294" y="70.9168" size="1.016" layer="25" rot="R180"/>
 <attribute name="VALUE" x="44.7548" y="69.596" size="1.016" layer="27" rot="R180"/>
@@
 <attribute name="VALUE" x="24.765" y="9.8298" size="1.016" layer="27"/>
 </element>
-<element name="THERM" library="testpad" library_urn="urn:adsk.eagle:library:385" package="TP20SQ" package3d_urn="urn:adsk.eagle:package:27980/1" value="TPSQTP20SQ" x="41.91" y="80.645" smashed="yes">
-<attribute name="NAME" x="39.894" y="78.5454" size="0.8128" layer="25"/>
-<attribute name="TP_SIGNAL_NAME" value="" x="41.91" y="78.105" size="1" layer="37"/>
+<element name="R2" library="resistor" library_urn="urn:adsk.eagle:library:348" package="R0805" package3d_urn="urn:adsk.eagle:package:23553/2" value="0" x="41.4528" y="77.8002" smashed="yes" rot="R270">
+<attribute name="NAME" x="42.5704" y="77.9018" size="1.016" layer="25"/>
+<attribute name="VALUE" x="42.5704" y="76.581" size="1.016" layer="27"/>
 </element>
 </elements>
@@
 <contactref element="LITHIUM-2" pad="V_AMP2"/>
 <contactref element="LITHIUM-2" pad="V_AMP1"/>
-<polygon width="0.1524" layer="1" thermals="no">
+<polygon width="0.2032" layer="1" thermals="no">
 <vertex x="89.535" y="65.024"/>
 <vertex x="89.535" y="61.976"/>
 <vertex x="89.535" y="59.69"/>
-<vertex x="37.465" y="59.69"/>
-<vertex x="37.465" y="66.04"/>
+<vertex x="38.1" y="59.69"/>
+<vertex x="38.1" y="66.04"/>
 <vertex x="89.535" y="66.04"/>
 </polygon>
@@
 <wire x1="42.545" y1="26.482" x2="40.097" y2="26.482" width="0.762" layer="1"/>
 <wire x1="40.097" y1="26.482" x2="39.585" y2="25.97" width="0.762" layer="1"/>
-<wire x1="42.545" y1="26.482" x2="42.545" y2="25.1714" width="0.762" layer="1"/>
-<via x="42.545" y="25.1714" extent="1-16" drill="0.508"/>
+<wire x1="42.545" y1="26.482" x2="42.545" y2="25.0952" width="0.762" layer="1"/>
+<via x="42.545" y="25.0952" extent="1-16" drill="0.508"/>
 <wire x1="39.585" y1="67.72" x2="39.585" y2="67.371" width="1.397" layer="1"/>
 <wire x1="39.585" y1="67.371" x2="42.418" y2="67.371" width="1.397" layer="1"/>
@@
 <wire x1="42.0878" y1="71.0946" x2="39.7096" y2="71.0946" width="1.524" layer="1"/>
 <wire x1="39.7096" y1="71.0946" x2="39.585" y2="70.97" width="1.524" layer="1"/>
+<contactref element="R2" pad="2"/>
+<wire x1="41.4528" y1="76.8502" x2="41.4528" y2="75.184" width="1.27" layer="1"/>
+<via x="41.4528" y="75.184" extent="1-16" drill="0.8382"/>
 </signal>
 <signal name="GPS_TX">
@@
 <contactref element="LITHIUM-2" pad="THERM2"/>
 <contactref element="LITHIUM-2" pad="THERM3"/>
-<polygon width="0.1524" layer="1" thermals="no">
+<polygon width="0.2032" layer="1" thermals="no">
 <vertex x="0" y="90.17"/>
 <vertex x="10.16" y="90.17"/>
@@
 <vertex x="0" y="34.29"/>
 </polygon>
-<polygon width="0.1524" layer="16" thermals="no">
+<polygon width="0.2032" layer="16" thermals="no">
 <vertex x="0" y="90.17"/>
 <vertex x="10.16" y="90.17"/>
@@
 <vertex x="0" y="0"/>
 </polygon>
-<contactref element="THERM" pad="TP"/>
 <contactref element="U$1" pad="MNT1"/>
+<contactref element="R2" pad="1"/>
 </signal>
 </signals>
